Commit message: Change all dashes in naes to underscores.
The move_group planner does not work with dashes in the names.

Karl D. Hansen <kdh@es.aau.dk>

File: robots/davinci_description.URDF (robot description, URDF)
Before this commit: robot davinci_description, 17 links, 16 joints
Links:
- removed link p4-arm-base
- removed link p4-arm1
- removed link p4-arm2
- removed link p4-arm3
- removed link p4-arm4
- removed link p4-hand1
- removed link p4-hand2
- removed link p4-hand3
- removed link p4-hand4
- removed link p4-hand4b
- removed link p4-hand5
- removed link p4-instrument-head
- removed link p4-instrument-house
- removed link p4-instrument-jawbone-left
- removed link p4-instrument-jawbone-right
- removed link p4-instrument-neck
- added link p4_arm1, mass 12.0042352614557; collision mesh filename=package://davinci_description/meshes/p4-arm1.STL; visual mesh filename=package://davinci_description/meshes/p4-arm1.STL
- added link p4_arm2, mass 7.45119488647257; collision mesh filename=package://davinci_description/meshes/p4-arm2.STL; visual mesh filename=package://davinci_description/meshes/p4-arm2.STL
- added link p4_arm3, mass 2.6382273355906; collision mesh filename=package://davinci_description/meshes/p4-arm3.STL; visual mesh filename=package://davinci_description/meshes/p4-arm3.STL
- added link p4_arm4, mass 1.95333539219675; collision mesh filename=package://davinci_description/meshes/p4-arm4.STL; visual mesh filename=package://davinci_description/meshes/p4-arm4.STL
- added link p4_arm_base, mass 4.57690792902629; collision mesh filename=package://davinci_description/meshes/p4-arm-base.STL; visual mesh filename=package://davinci_description/meshes/p4-arm-base.STL
- added link p4_hand1, mass 0.621071194298928; collision mesh filename=package://davinci_description/meshes/p4-hand1.STL; visual mesh filename=package://davinci_description/meshes/p4-hand1.STL
- added link p4_hand2, mass 0.282965703322585; collision mesh filename=package://davinci_description/meshes/p4-hand2.STL; visual mesh filename=package://davinci_description/meshes/p4-hand2.STL
- added link p4_hand3, mass 1.10069000101175; collision mesh filename=package://davinci_description/meshes/p4-hand3.STL; visual mesh filename=package://davinci_description/meshes/p4-hand3.STL
- added link p4_hand4, mass 0.447187973747169; collision mesh filename=package://davinci_description/meshes/p4-hand4.STL; visual mesh filename=package://davinci_description/meshes/p4-hand4.STL
- added link p4_hand4b, mass 0.447187973747169; collision mesh filename=package://davinci_description/meshes/p4-hand4.STL; visual mesh filename=package://davinci_description/meshes/p4-hand4.STL
- added link p4_hand5, mass 1.36700413065379; collision mesh filename=package://davinci_description/meshes/p4-hand5.STL; visual mesh filename=package://davinci_description/meshes/p4-hand5.STL
- added link p4_instrument_head, mass 0.000234269246654977; collision mesh filename=package://davinci_description/meshes/p4-instrument-head.STL; visual mesh filename=package://davinci_description/meshes/p4-instrument-head.STL
- added link p4_instrument_house, mass 0.160905448095996; collision mesh filename=package://davinci_description/meshes/p4-instrument-house.STL; visual mesh filename=package://davinci_description/meshes/p4-instrument-house.STL
- added link p4_instrument_jawbone-left, mass 4.72823027124423E-05; collision mesh filename=package://davinci_description/meshes/p4-instrument-jawbone-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; visual mesh filename=package://davinci_description/meshes/p4-instrument-jawbone-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
- added link p4_instrument_jawbone-right, mass 4.72823027124613E-05; collision mesh filename=package://davinci_description/meshes/p4-instrument-jawbone-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; visual mesh filename=package://davinci_description/meshes/p4-instrument-jawbone-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
- added link p4_instrument_neck, mass 0.0232510537357557; collision mesh filename=package://davinci_description/meshes/p4-instrument-neck.STL; visual mesh filename=package://davinci_description/meshes/p4-instrument-neck.STL
Joints:
- removed joint p4-arm-elevation
- removed joint p4-arm-roll1
- removed joint p4-arm-yaw1
- removed joint p4-arm-yaw2
- removed joint p4-arm-yaw3
- removed joint p4-arm-yaw4
- removed joint p4-hand-pitch
- removed joint p4-hand-pitch2
- removed joint p4-hand-pitch2b
- removed joint p4-hand-pitch3
- removed joint p4-hand-roll
- removed joint p4-instrument-jaw-left
- removed joint p4-instrument-jaw-right
- removed joint p4-instrument-pitch
- removed joint p4-instrument-roll
- removed joint p4-instrument-slide
- added joint p4_arm_elevation: type prismatic, parent base_link, child p4_arm_base, origin xyz=0 0 0 rpy=0 0 0, axis 0 0 1, limit lower=0 upper=1 effort=1 velocity=1
- added joint p4_arm_roll1: type revolute, parent p4_arm3, child p4_arm4, origin xyz=0.0569999999999999 0 0.19825 rpy=-2.72945570336682E-16 2.973835489358E-19 -9.62964972193618E-35, axis -1 0 0, limit lower=-1.5708 upper=1.5708 effort=1 velocity=1
- added joint p4_arm_yaw1: type revolute, parent p4_arm_base, child p4_arm1, origin xyz=0.186 0 0.5544 rpy=3.1416 0 1.5708, axis 0 0 1, limit lower=-1.5708 upper=1.5708 effort=1 velocity=1
- added joint p4_arm_yaw2: type revolute, parent p4_arm1, child p4_arm2, origin xyz=0 0.58285 0 rpy=-3.14159265358979 1.24808068980918E-16 1.5707963267949, axis 0 0 -1, limit lower=-2.8 upper=2.8 effort=1 velocity=1
- added joint p4_arm_yaw3: type revolute, parent p4_arm2, child p4_arm3, origin xyz=0.47985 0 -0.001 rpy=-4.41862941934989E-22 2.30317389564735E-22 -1.30104260698261E-18, axis 0 0 -1, limit lower=-2.8 upper=2.8 effort=1 velocity=1
- added joint p4_arm_yaw4: type revolute, parent p4_arm4, child p4_hand1, origin xyz=0.35225 0 -0.117 rpy=3.22833053553567E-17 2.04577519985781E-18 8.67361737988404E-19, axis 0 0 1, limit lower=-2.8 upper=2.8 effort=1 velocity=1
- added joint p4_hand_pitch: type revolute, parent p4_hand2, child p4_hand3, origin xyz=0 0 0 rpy=3.42136669122662E-16 -0.288812097817057 -1.17706479711569E-17, axis 0 1 0, limit lower=-0.8 upper=1.0 effort=1 velocity=1
- added joint p4_hand_pitch2: type continuous, parent p4_hand3, child p4_hand4, origin xyz=0.0108229214977171 0 0.186426149539229 rpy=3.14159265358979 0.288812097814836 9.64324654702006E-17, axis 0 1 0, mimic joint=p4_hand_pitch
- added joint p4_hand_pitch2b: type continuous, parent p4_hand3, child p4_hand4b, origin xyz=0 0 0.15 rpy=3.14159265358979 0.288812097814836 9.64324654702006E-17, axis 0 1 0, mimic joint=p4_hand_pitch
- added joint p4_hand_pitch3: type continuous, parent p4_hand4, child p4_hand5, origin xyz=0.52 0 0 rpy=3.14159265358979 -2.22109682611874E-12 6.08324503520137E-16, axis 0 -1 0, mimic joint=p4_hand_pitch multiplier=-1
- added joint p4_hand_roll: type revolute, parent p4_hand1, child p4_hand2, origin xyz=-0.0424999999999998 0 0.160999999999999 rpy=0 1.22464679914735E-16 0, axis 1 0 0, limit lower=-1.5708 upper=1.5708 effort=1 velocity=1
- added joint p4_instrument_jaw-left: type continuous, parent p4_instrument_head, child p4_instrument_jawbone-left, origin xyz=0 0 0.00900000000000001 rpy=1.5707963267949 1.5707963267949 0, axis 0 0 1
- added joint p4_instrument_jaw-right: type continuous, parent p4_instrument_head, child p4_instrument_jawbone-right, origin xyz=0 0 0.00900000000000001 rpy=1.5707963267949 1.5707963267949 0, axis 0 0 -1
- added joint p4_instrument_pitch: type continuous, parent p4_instrument_neck, child p4_instrument_head, origin xyz=0 0 0.177 rpy=0 0 0, axis 1 0 0
- added joint p4_instrument_roll: type continuous, parent p4_instrument_house, child p4_instrument_neck, origin xyz=0.0525000000003168 0 0 rpy=3.14159265358979 -1.45892264612837E-16 1.5707963267949, axis 0 0 1
- added joint p4_instrument_slide: type prismatic, parent p4_hand5, child p4_instrument_house, origin xyz=0 0 0 rpy=0 0 0, axis 0 0 -1, limit lower=0 upper=0.3 effort=1 velocity=1

Commit message: Change the rest of the names to dashes.
I forgot to change the names includeing jaw.

Signed-off-by: Karl Damkjær Hansen <kdh@es.aau.dk>

File: robots/davinci_description.URDF (robot description, URDF)
Before this commit: robot davinci_description, 17 links, 16 joints
Links:
- removed link p4_instrument_jawbone-left
- removed link p4_instrument_jawbone-right
- added link p4_instrument_jawbone_left, mass 4.72823027124423E-05; collision mesh filename=package://davinci_description/meshes/p4-instrument-jawbone-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; visual mesh filename=package://davinci_description/meshes/p4-instrument-jawbone-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
- added link p4_instrument_jawbone_right, mass 4.72823027124613E-05; collision mesh filename=package://davinci_description/meshes/p4-instrument-jawbone-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; visual mesh filename=package://davinci_description/meshes/p4-instrument-jawbone-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
Joints:
- removed joint p4_instrument_jaw-left
- removed joint p4_instrument_jaw-right
- added joint p4_instrument_jaw_left: type continuous, parent p4_instrument_head, child p4_instrument_jawbone_left, origin xyz=0 0 0.00900000000000001 rpy=1.5707963267949 1.5707963267949 0, axis 0 0 1
- added joint p4_instrument_jaw_right: type continuous, parent p4_instrument_head, child p4_instrument_jawbone_right, origin xyz=0 0 0.00900000000000001 rpy=1.5707963267949 1.5707963267949 0, axis 0 0 -1

Commit message: Include Christoffers modifications
Christoffer machined the davinci model to work with gazebo and moveit!
Things may not be pretty but they are working.

Signed-off-by: Karl Damkjær Hansen <kdh@es.aau.dk>

File: robots/davinci_description.URDF (robot description, URDF)
Before this commit: robot davinci_description, 17 links, 16 joints
Links:
- added link world
Joints:
- added joint fixed: type fixed, parent world, child base_link
- joint p4_hand_pitch2: mimic joint=p4_hand_pitch -> (none)
- joint p4_hand_pitch2b: mimic joint=p4_hand_pitch -> (none)
- joint p4_hand_pitch3: mimic joint=p4_hand_pitch multiplier=-1 -> (none)
- joint p4_instrument_slide: limit lower=0 upper=0.3 effort=1 velocity=1 -> lower=0 upper=1 effort=1 velocity=1
