Commit message: Modified xacro without passive joints

File: robots/davinci_link_macro.xacro (robot description, xacro)
@@ -4,5 +4,5 @@
   <xacro:unless value="${macros_included}">
     <xacro:property name="macros_included" value="true" />
-    <xacro:macro name="davinci_link" params="name color *block">
+    <xacro:macro name="davinci_link" params="name color">
       <link name="${name}">
         <visual>
@@ -23,5 +23,4 @@
           </geometry>
         </collision>
-        <xacro:insert_block name="block" />
       </link>
     </xacro:macro>

File: robots/instruments/needle_driver.xacro (robot description, xacro)
@@ -2,18 +2,4 @@
 <robot name="davinci" xmlns:xacro="http://www.ros.org/wiki/xacro">
   <link name="needle_driver_house">
-    <inertial>
-      <origin
-        xyz="0.0487926923825119 1.2425463059237E-09 0.303878514609369"
-        rpy="0 0 0" />
-      <mass
-        value="0.160905448095996" />
-      <inertia
-        ixx="0.000147992717312588"
-        ixy="-4.85204886997006E-13"
-        ixz="-2.43650182134419E-06"
-        iyy="0.000117219380395437"
-        iyz="-1.68887809351124E-11"
-        izz="5.63867712385493E-05" />
-    </inertial>
     <visual>
       <origin
@@ -38,19 +24,22 @@
     </collision>
   </link>
+  <joint name="p4_instrument_roll"
+    type="revolute">
+    <origin
+      xyz="0 0 0"
+      rpy="0 0 0" />
+    <parent
+      link="needle_driver_house" />
+    <child
+      link="needle_driver_neck" />
+    <axis
+      xyz="0 0 1" />
+    <limit
+      lower="-4.712"
+      upper="4.712"
+      effort="1"
+      velocity="1" />
+  </joint>
   <link name="needle_driver_neck">
-    <inertial>
-      <origin
-        xyz="1.88981532714125E-09 3.16376702613752E-10 -0.0401302981872702"
-        rpy="0 0 0" />
-      <mass
-        value="0.0232510537357557" />
-      <inertia
-        ixx="0.000357953997322209"
-        ixy="-1.09841765686305E-13"
-        ixz="7.75110601988088E-12"
-        iyy="0.000357954438471494"
-        iyz="1.3024211024653E-12"
-        izz="2.00399317932057E-07" />
-    </inertial>
     <visual>
       <origin
@@ -75,37 +64,22 @@
     </collision>
   </link>
-  <joint name="p4_instrument_roll"
+  <joint name="p4_instrument_pitch"
     type="revolute">
     <origin
-      xyz="0.0525000000003168 0 0"
-      rpy="3.14159265358979 -1.45892264612837E-16 1.5707963267949" />
+      xyz="0 0 0"
+      rpy="0 1.5708 0" />
     <parent
-      link="needle_driver_house" />
+      link="needle_driver_neck" />
     <child
-      link="needle_driver_neck" />
+      link="needle_driver_head" />
     <axis
       xyz="0 0 1" />
     <limit
-      lower="-4.712"
-      upper="4.712"
+      lower="-1.5"
+      upper="1.5"
       effort="1"
       velocity="1" />
-    <dynamics damping="0"/>
   </joint>
   <link name="needle_driver_head">
-    <inertial>
-      <origin
-        xyz="2.82477802579071E-06 -3.6037163499536E-05 0.00301833175193345"
-        rpy="0 0 0" />
-      <mass
-        value="0.000234269246654977" />
-      <inertia
-        ixx="2.57553175127649E-09"
-        ixy="-1.7088879166498E-11"
-        ixz="4.50036079768168E-13"
-        iyy="2.37501406336667E-09"
-        iyz="-1.57952093810846E-11"
-        izz="1.24185526283754E-09" />
-    </inertial>
     <visual>
       <origin
@@ -130,37 +104,22 @@
     </collision>
   </link>
-  <joint name="p4_instrument_pitch"
+  <joint name="p4_instrument_jaw_right"
     type="revolute">
     <origin
-      xyz="0 0 0.177"
-      rpy="0 0 0" />
+      xyz="0.009 0 0"
+      rpy="-1.5708 0 0" />
     <parent
-      link="needle_driver_neck" />
+      link="needle_driver_head" />
     <child
-      link="needle_driver_head" />
+      link="needle_driver_jawbone_right" />
     <axis
-      xyz="-1 0 0" />
+      xyz="0 0 1" />
     <limit
-      lower="-1.5"
-      upper="1.5"
+      lower="-1.8"
+      upper="1.8"
       effort="1"
       velocity="1" />
-    <dynamics damping="0"/>
   </joint>
   <link name="needle_driver_jawbone_right">
-    <inertial>
-      <origin
-        xyz="-0.00211142946935594 0.000167266219560752 -0.000657389690164489"
-        rpy="0 0 0" />
-      <mass
-        value="4.72823027124423E-05" />
-      <inertia
-        ixx="7.07960996815586E-11"
-        ixy="-3.38178696144901E-11"
-        ixz="-5.27585618542085E-11"
-        iyy="4.60880145483977E-10"
-        iyz="5.64458037529414E-12"
-        izz="4.87285720312733E-10" />
-    </inertial>
     <visual>
       <origin
@@ -185,37 +144,5 @@
     </collision>
   </link>
-  <joint name="p4_instrument_jaw_right"
-    type="revolute">
-    <origin
-      xyz="0 0 0.00900000000000001"
-      rpy="1.5707963267949 1.5707963267949 0" />
-    <parent
-      link="needle_driver_head" />
-    <child
-      link="needle_driver_jawbone_right" />
-    <axis
-      xyz="0 0 1" />
-    <limit
-      lower="-1.8"
-      upper="1.8"
-      effort="1"
-      velocity="1" />
-    <dynamics damping="0"/>
-  </joint>
   <link name="needle_driver_jawbone_left">
-    <inertial>
-      <origin
-        xyz="-0.00211142946935583 0.000167266219581923 -0.000749389690795965"
-        rpy="0 0 0" />
-      <mass
-        value="4.72823027124613E-05" />
-      <inertia
-        ixx="7.07960996815865E-11"
-        ixy="-3.38178696144904E-11"
-        ixz="-5.27585618541835E-11"
-        iyy="4.60880145483901E-10"
-        iyz="5.64458037527874E-12"
-        izz="4.87285720312658E-10" />
-    </inertial>
     <visual>
       <origin
@@ -243,6 +170,6 @@
     type="revolute">
     <origin
-      xyz="0 0 0.00900000000000001"
-      rpy="1.5707963267949 1.5707963267949 0" />
+      xyz="0.009 0 0"
+      rpy="-1.5708 0 0" />
     <parent
       link="needle_driver_head" />
@@ -250,5 +177,5 @@
       link="needle_driver_jawbone_left" />
     <axis
-      xyz="0 0 -1" />
+      xyz="0 0 1" />
     <limit
       lower="-1.8"
@@ -256,5 +183,4 @@
       effort="1"
       velocity="1" />
-    <dynamics damping="0" friction="0.1"/>
   </joint>
 </robot>

File: robots/p4_arm.xacro (robot description, xacro)
@@ -12,14 +12,4 @@
       <material name="surgical gray"/>
     </visual>
-    <inertial>
-      <origin
-        xyz="0.1602 0 0.4561"
-        rpy="0 0 0" />
-      <mass value="2" />
-    <inertia
-      ixx="1" ixy="0" ixz="0"
-              iyy="1" iyz="0"
-                      izz="1" />
-    </inertial>
     <collision>
       <origin
@@ -38,6 +28,6 @@
       link="p4_arm1"/>
     <origin
-      xyz="0.186 0 0.5544"
-      rpy="3.1416 0 1.5708" />
+      xyz="0.198 0 0"
+      rpy="0 0 0" />
     <axis
       xyz="0 0 1"/>
@@ -47,26 +37,11 @@
       effort="1"
       velocity="1" />
-    <dynamics
-      damping="0.7"/>
   </joint>
-  <xacro:davinci_link name="p4_arm1"
-    color="surgical gray">
-    <inertial>
-    <origin
-      xyz="0 0.2529 -0.0998"
-      rpy="0 0 0" />
-    <mass
-      value="5" />
-    <inertia
-      ixx="1" ixy="0" ixz="0"
-              iyy="1" iyz="0"
-                      izz="1" />
-    </inertial>
-  </xacro:davinci_link>
+  <xacro:davinci_link name="p4_arm1" color="surgical gray"/>
   <joint name="p4_arm_yaw2"
     type="revolute">
     <origin
-      xyz="0 0.58285 0"
-      rpy="-3.14159 0 1.5707" />
+      xyz="0.582 0 0"
+      rpy="0 0 0" />
     <parent
       link="p4_arm1" />
@@ -74,5 +49,5 @@
       link="p4_arm2" />
     <axis
-      xyz="0 0 -1" />
+      xyz="0 0 1" />
     <limit
       lower="-2.8"
@@ -83,23 +58,10 @@
       damping="0.7"/>
   </joint>
-  <xacro:davinci_link name="p4_arm2"
-    color="surgical gray">
-    <inertial>
-      <origin
-        xyz="0.2247 0 -0.0850"
-        rpy="0 0 0" />
-      <mass
-        value="7" />
-       <inertia
-        ixx="1" ixy="0" ixz="0"
-                iyy="1" iyz="0"
-                        izz="1" />
-    </inertial>
-  </xacro:davinci_link>
+  <xacro:davinci_link name="p4_arm2" color="surgical gray" />
   <joint name="p4_arm_yaw3"
     type="revolute">
     <origin
-      xyz="0.47985 0 -0.001"
-      rpy="-4.41862941934989E-22 2.30317389564735E-22 -1.30104260698261E-18" />
+      xyz="0.435 0 0"
+      rpy="0 0 0" />
     <parent
       link="p4_arm2" />
@@ -107,5 +69,5 @@
       link="p4_arm3" />
     <axis
-      xyz="0 0 -1" />
+      xyz="0 0 1" />
     <limit
       lower="-2.8"
@@ -116,23 +78,10 @@
       damping="0"/>
   </joint>
-  <xacro:davinci_link name="p4_arm3"
-    color="surgical gray">
-    <inertial>
-      <origin
-        xyz="-0.0267 0 0.1459"
-        rpy="0 0 0" />
-      <mass
-        value="2" />
-      <inertia
-        ixx="1" ixy="0" ixz="0"
-                iyy="1" iyz="0"
-                        izz="1" />
-    </inertial>
-  </xacro:davinci_link>
+  <xacro:davinci_link name="p4_arm3" color="surgical gray" />
   <joint name="p4_arm_roll1"
     type="revolute">
     <origin
-      xyz="0.0570 0 0.1982"
-      rpy="0 0 0" />
+      xyz="0 0 0"
+      rpy="0 1.5708 0" />
     <parent
       link="p4_arm3" />
@@ -140,5 +89,5 @@
       link="p4_arm4" />
     <axis
-      xyz="-1 0 0" />
+      xyz="0 0 1" />
     <limit
       lower="-1.5708"
@@ -146,26 +95,11 @@
       effort="1"
       velocity="1" />
-    <dynamics
-      damping="0"/>
   </joint>
-  <xacro:davinci_link name="p4_arm4"
-    color="surgical gray">
-    <inertial>
-      <origin
-        xyz="0.1739 0 -0.1235"
-        rpy="0 0 0" />
-      <mass
-        value="2" />
-      <inertia
-        ixx="1" ixy="0" ixz="0"
-                iyy="1" iyz="0"
-                        izz="1" />
-    </inertial>
-  </xacro:davinci_link>
+  <xacro:davinci_link name="p4_arm4" color="surgical gray" />
   <joint name="p4_arm_yaw4"
     type="revolute">
     <origin
-      xyz="0.3522 0 -0.117"
-      rpy="0 0 0" />
+      xyz="0 0 0.412"
+      rpy="0 -1.5708 0" />
     <parent
       link="p4_arm4" />
@@ -179,6 +113,4 @@
       effort="1"
       velocity="1" />
-    <dynamics
-      damping="0"/>
   </joint>
 </robot>

File: robots/remote_center_manipulator.xacro (robot description, xacro)
@@ -2,43 +2,16 @@
 <robot name="davinci" xmlns:xacro="http://www.ros.org/wiki/xacro">
   <xacro:include filename="$(find davinci_description)/robots/davinci_link_macro.xacro" />
-  <xacro:davinci_link name="p4_rcm_base"
-    color="slate">
-    <inertial>
-      <origin
-        xyz="-0.141021 0 0.066384"
-        rpy="0 0 0" />
-      <mass
-        value="0.6" />
-      <inertia
-        ixx="1" ixy="0" ixz="0"
-                iyy="1" iyz="0"
-                        izz="1" />
-    </inertial>
-  </xacro:davinci_link>
-  <xacro:davinci_link name="p4_rcm_pivot_plate"
-    color="slate">
-    <inertial>
-      <origin
-        xyz="-0.0349 0.0169 -0.0063"
-        rpy="0 0 0" />
-      <mass
-      value="0.2829" />
-      <inertia
-        ixx="1" ixy="0" ixz="0"
-                iyy="1" iyz="0"
-                        izz="1" />
-    </inertial>
-  </xacro:davinci_link>
+  <xacro:davinci_link name="p4_rcm_base" color="slate" />
   <joint name="p4_hand_roll"
     type="revolute">
     <origin
-      xyz="-0.0425 0 0.1610"
-      rpy="0 0 0" />
+      xyz="0.482 0 0.047"
+      rpy="0 1.5708 0" />
     <parent
       link="p4_rcm_base" />
     <child
-      link="p4_rcm_pivot_plate" />
+      link="rcm_vitual0" />
     <axis
-      xyz="1 0 0" />
+      xyz="0 0 1" />
     <limit
       lower="-1.5708"
@@ -46,32 +19,17 @@
       effort="1"
       velocity="1" />
-    <dynamics
-      damping="0"/>
   </joint>
-  <xacro:davinci_link name="p4_rcm_parallelogram_base"
-    color="slate">
-    <inertial>
-      <origin
-        xyz="-0.0085 0 -0.0484"
-        rpy="0 0 0" />
-      <mass
-        value="1" />
-      <inertia
-        ixx="1" ixy="0" ixz="0"
-                iyy="1" iyz="0"
-                        izz="1" />
-    </inertial>
-  </xacro:davinci_link>
+  <link name="rcm_vitual0" />
   <joint name="p4_hand_pitch"
     type="revolute">
     <origin
       xyz="0 0 0"
-      rpy="0 -0.2888 0" />
+      rpy="1.5708 0 0" />
     <parent
-      link="p4_rcm_pivot_plate" />
+      link="rcm_vitual0" />
     <child
-      link="p4_rcm_parallelogram_base" />
+      link="rcm_vitual1" />
     <axis
-      xyz="0 -1 0" />
+      xyz="0 0 1" />
     <limit
       lower="-0.8"
@@ -79,77 +37,13 @@
       effort="1"
       velocity="1" />
-    <dynamics damping="0"/>
   </joint>
-  <xacro:davinci_link name="p4_rcm_parallelogram_upper_bar"
-    color="slate">
-    <inertial>
-      <origin
-        xyz="0.263815 0 0"
-        rpy="0 0 0" />
-      <mass
-        value="0.447188" />
-      <inertia
-        ixx="1" ixy="0" ixz="0"
-                iyy="1" iyz="0"
-                        izz="1" />
-    </inertial>
-  </xacro:davinci_link>
-  <joint name="p4_rcm_upper_bar_base_joint"
-    type="continuous">
-    <origin
-      xyz="0.0108 0 0.1864"
-      rpy="3.14159 0.28881 0" />
-    <parent
-      link="p4_rcm_parallelogram_base" />
-    <child
-      link="p4_rcm_parallelogram_upper_bar" />
-    <axis
-      xyz="0 1 0" />
-    <mimic
-      joint="p4_hand_pitch"
-      multiplier="-1.0"
-      offset="0.0" />
-    <dynamics
-      damping="0"/>
-  </joint>
-  <xacro:davinci_link name="p4_rcm_instrument_holder"
-    color="slate">
-    <inertial>
-      <origin
-        xyz="0.010300 0 0.115001"
-        rpy="0 0 0" />
-      <mass
-        value="1.367004" />
-      <inertia
-        ixx="1" ixy="0" ixz="0"
-                iyy="1" iyz="0"
-                        izz="1" />
-    </inertial>
-  </xacro:davinci_link>
-  <joint name="p4_rcm_instrument_holder_upper_bar_joint"
-    type="continuous">
-    <origin
-      xyz="0.52 0 0"
-      rpy="3.141593 0 0" />
-    <parent
-      link="p4_rcm_parallelogram_upper_bar" />
-    <child
-      link="p4_rcm_instrument_holder" />
-    <axis
-      xyz="0 -1 0" />
-    <mimic
-      joint="p4_hand_pitch"
-      multiplier="1.0"
-      offset="0.0" />
-    <dynamics
-      damping="0"/>
-  </joint>
+  <link name="rcm_vitual1" />
   <joint name="p4_instrument_slide"
     type="prismatic">
     <origin
-      xyz="0 0 -0.12"
-      rpy="0 0 0" />
+      xyz="0.097 0 0"
+      rpy="0 -1.5708 0" />
     <parent
-      link="p4_rcm_instrument_holder" />
+      link="rcm_vitual1" />
     <child
       link="needle_driver_house" />
@@ -161,5 +55,4 @@
       effort="1"
       velocity="1" />
-    <dynamics damping="0"/>
   </joint>
 </robot>

File: robots/tower.xacro (robot description, xacro)
@@ -2,22 +2,10 @@
 <robot name="davinci" xmlns:xacro="http://www.ros.org/wiki/xacro">
   <xacro:include filename="$(find davinci_description)/robots/davinci_link_macro.xacro" />
-  <xacro:davinci_link name="base_link"
-    color="surgical gray">
-    <inertial>
-      <origin
-        xyz="0 0 0"
-        rpy="0 0 0" />
-      <mass value="100" />
-    <inertia
-      ixx="1" ixy="0" ixz="0"
-              iyy="1" iyz="0"
-                      izz="1" />
-    </inertial>
-  </xacro:davinci_link>
+  <xacro:davinci_link name="base_link" color="surgical gray"/>
   <joint name="p4_arm_elevation" type="prismatic">
     <parent link="base_link"/>
     <child link="p4_arm_base"/>
     <origin
-      xyz="0 0 0"
+      xyz="0 0 0.998"
       rpy="0 0 0" />
     <axis xyz="0 0 1"/>
