Commit message: Fix model roll, pitch and yaw
Some of the rotations were in the wrong direction.

Signed-off-by: Karl Damkjær Hansen <kdh@es.aau.dk>

File: robots/instruments/needle_driver.xacro (robot description, xacro)
@@ -140,5 +140,5 @@
       link="needle_driver_head" />
     <axis
-      xyz="1 0 0" />
+      xyz="-1 0 0" />
     <limit
       lower="-1.5"
@@ -148,5 +148,5 @@
     <dynamics damping="0"/>
   </joint>
-  <link name="needle_driver_jawbone_left">
+  <link name="needle_driver_jawbone_right">
     <inertial>
       <origin
@@ -185,5 +185,5 @@
     </collision>
   </link>
-  <joint name="p4_instrument_jaw_left"
+  <joint name="p4_instrument_jaw_right"
     type="revolute">
     <origin
@@ -193,5 +193,5 @@
       link="needle_driver_head" />
     <child
-      link="needle_driver_jawbone_left" />
+      link="needle_driver_jawbone_right" />
     <axis
       xyz="0 0 1" />
@@ -203,5 +203,5 @@
     <dynamics damping="0"/>
   </joint>
-  <link name="needle_driver_jawbone_right">
+  <link name="needle_driver_jawbone_left">
     <inertial>
       <origin
@@ -224,5 +224,5 @@
       <geometry>
         <mesh
-          filename="package://davinci_description/meshes/instruments/needle_driver_jawbone_right.stl" />
+          filename="package://davinci_description/meshes/instruments/needle_driver_jawbone_left.stl" />
       </geometry>
       <material
@@ -236,9 +236,9 @@
       <geometry>
         <mesh
-          filename="package://davinci_description/meshes/instruments/needle_driver_jawbone_right.stl" />
-      </geometry>
-    </collision>
-  </link>
-  <joint name="p4_instrument_jaw_right"
+          filename="package://davinci_description/meshes/instruments/needle_driver_jawbone_left.stl" />
+      </geometry>
+    </collision>
+  </link>
+  <joint name="p4_instrument_jaw_left"
     type="revolute">
     <origin
@@ -248,5 +248,5 @@
       link="needle_driver_head" />
     <child
-      link="needle_driver_jawbone_right" />
+      link="needle_driver_jawbone_left" />
     <axis
       xyz="0 0 -1" />

File: robots/remote_center_manipulator.xacro (robot description, xacro)
@@ -6,8 +6,8 @@
     <inertial>
       <origin
-        xyz="-0.141020957350944 1.21214233081955E-17 0.0663841857186647"
+        xyz="-0.141021 0 0.066384"
         rpy="0 0 0" />
       <mass
-        value="0.621071194298928" />
+        value="0.6" />
       <inertia
         ixx="1" ixy="0" ixz="0"
@@ -73,5 +73,5 @@
       link="p4_rcm_parallelogram_base" />
     <axis
-      xyz="0 1 0" />
+      xyz="0 -1 0" />
     <limit
       lower="-0.8"
@@ -108,5 +108,5 @@
     <mimic
       joint="p4_hand_pitch"
-      multiplier="1.0"
+      multiplier="-1.0"
       offset="0.0" />
     <dynamics
@@ -140,5 +140,5 @@
     <mimic
       joint="p4_hand_pitch"
-      multiplier="-1.0"
+      multiplier="1.0"
       offset="0.0" />
     <dynamics
@@ -148,5 +148,5 @@
     type="prismatic">
     <origin
-      xyz="0 0 0"
+      xyz="0 0 -0.12"
       rpy="0 0 0" />
     <parent
@@ -155,8 +155,8 @@
       link="needle_driver_house" />
     <axis
-      xyz="0 0 -1" />
+      xyz="0 0 1" />
     <limit
-      lower="0"
-      upper="0.3"
+      lower="-0.12"
+      upper="0.12"
       effort="1"
       velocity="1" />
